Commit message: more natural roles for transmission components

File: examples/single_dynamixel/description/ros2_control.xacro (robot description, xacro)
@@ -40,6 +40,6 @@
         <transmission name="axis_trans">
             <plugin>transmission_interface/SimpleTransmission</plugin>
-            <actuator name="axis_dynamixel" role="axis_dynamixel"/>
-            <joint name="axis" role="axis">
+            <actuator name="axis_dynamixel" role="actuator"/>
+            <joint name="axis" role="joint">
                 <mechanical_reduction>1.0</mechanical_reduction>
                 <offset>0.0</offset>
